File: LedMatrix.sch (KiCad schematic (older format))
At the start: 151 parts

Commit message: Add PCB file
Parts:
- LED01, LED02, LED03, LED031, LED04, LED041, LED05, LED0512, LED06, LED07, LED08, LED09, LED10, LED101, LED102, LED11, LED12, LED13, LED14, LED15, LED151, LED16, LED17, LED18, LED19, LED21, LED22, LED23, LED24, LED26, LED27, LED28, LED29, LED30, LED301, LED302, LED31, LED32, LED33, LED34, LED36, LED37, LED38, LED39, LED41, LED42, LED43, LED44, LED46, LED47, LED48, LED49, LED50, LED51, LED52, LED53, LED54, LED55, LED552, LED56, LED57, LED58, LED59, LED60, LED601, LED602, LED61, LED62, LED63, LED64, LED641, LED65, LED6512, LED66, LED661, LED67, LED68, LED681, LED682, LED69, LED691, LED692, LED70, LED7012: footprint (none) -> mx1a-led:MX1A-led
- LR05, LR09, LR1, LR10, LR11, LR12, LR13, LR14, LR15, LR16, LR17, LR18, LR19, LR2, LR21, LR22, LR23, LR24, LR26, LR27, LR28, LR29, LR3, LR30, LR31, LR32, LR33, LR34, LR36, LR37, LR38, LR4, LR41, LR42, LR43, LR44, LR46, LR47, LR48, LR49, LR50, LR51, LR52, LR53, LR54, LR55, LR56, LR57, LR58, LR59, LR6, LR60, LR61, LR62, LR63, LR64, LR65, LR66, LR67, LR68, LR69, LR7, LR70, LR8: footprint (none) -> SM0805:SM0805
- LR39: renamed from LED39; footprint (none) -> SM0805:SM0805
- Q1: renamed from Q?; footprint (none) -> sot23:sot23_handsoldering
- R1: renamed from R?; footprint (none) -> SM0805:SM0805
Connections:
- wire segments 414 -> 245

Commit message: add new footprints
Parts:
- LED01, LED02, LED03, LED031, LED04, LED041, LED05, LED0512, LED06, LED07, LED08, LED09, LED10, LED101, LED102, LED11, LED12, LED13, LED14, LED15, LED151, LED16, LED17, LED18, LED19, LED21, LED22, LED23, LED24, LED26, LED27, LED28, LED29, LED30, LED301, LED302, LED31, LED32, LED33, LED34, LED36, LED37, LED38, LED39, LED41, LED42, LED43, LED44, LED46, LED47, LED48, LED49, LED50, LED51, LED52, LED53, LED54, LED55, LED552, LED56, LED57, LED58, LED59, LED60, LED601, LED602, LED61, LED62, LED63, LED64, LED641, LED65, LED6512, LED66, LED661, LED67, LED68, LED681, LED682, LED69, LED691, LED692, LED70, LED7012: symbol LED -> LED-RESCUE-keyboard
