File: keyboard.kicad_pcb (KiCad board)
At the start: 2 copper layers, 285 x 94.6 mm, 321 parts, among them Q1 MOS_P

Commit message: add alps switch compatibility
Parts:
- S01, S02, S04, S041, S05, S06, S07, S08, S09, S10, S11, S12, S13, S14, S15, S16, S17, S18, S19, S21, S22, S23, S24, S26, S27, S28, S29, S30, S31, S32, S33, S34, S36, S37, S38, S39, S41, S42, S43, S44, S46, S47, S48, S49, S50, S51, S52, S53, S54, S55, S56, S57, S58, S59, S60, S61, S62, S63, S64, S65, S66, S661, S67, S68, S682, S69, S70: footprint MX1A-b -> mx_alps:Mx_Alps_100
- S03: footprint mx1a:MX1A -> mx_alps:Mx_Alps_100
- S031: footprint mx1a:MX1A -> mx1a:MX1A-b
- S0512, S101, S102, S151, S301, S302, S552, S601, S602, S641, S6512, S681, S691, S692, S7012: footprint MX1A-b -> mx1a:MX1A-b
